File: G0.sch (EAGLE design)
At the start: 0 parts

Commit message: Rev0
Parts:
- added AE1: ANT3216A063R2400A, ANT3216A063R2400A:ANT3216A063R2400A
- added BTN1, BTN2: TL3780AF330QG, TL3780AF330QG:TL3780AF330QG
- added C1, C2: 20pF/±2%, SparkFun-Capacitors:0.1UF-0402-16V-10%
- added C3: 5.6pF, SparkFun-Capacitors:0.1UF-0603-100V-10%
- added C4: 10pF, SparkFun-Capacitors:1.0UF-0805-25V-10%
- added C5: 12pF, SparkFun-Capacitors:0.1UF-0402-16V-10%
- added J1: USB4080-03-A_REVA1, USB4080-03-A_REVA1:USB4080-03-A_REVA1
- added J2: USB4085-GF-A_REVB, USB4085-GF-A_REVB:USB4085-GF-A_REVB
- added J3: SFV24R-3STBE1HLF, SFV24R-3STBE1HLF:SFV24R-3STBE1HLF
- added L1: 24nH/±2%/500mA, SparkFun-Coils:INDUCTOR-0603-33NH
- added L2, L3: 0.8nH, SparkFun-Coils:INDUCTOR-0603-15NH
- added Q1: FS8205A, FS8205A:FS8205A
- added R1, R11, R12, R13, R14, R17, R2, R3, R4, R5: 0, SparkFun-Resistors:0OHM-0603-1/10W
- added R10, R15, R16, R6, R7, R8, R9: 5.1k, SparkFun-Resistors:5.1KOHM5.1KOHM-0603-1/10W-1%
- added U$1: TP4056, TP4056:TP4056
- added U1: ESP32-S3R8, ESP32-S3:ESP32-S3
- added U2: W25Q128JVSIQ, W25Q128JVSIQ:W25Q128JVSIQ
- added U3: CP2102N-A01-GQFN28, CP2102N-A01-GQFN28:CP2102N-A01-GQFN28
- added U4: DW01A, DW01A:DW01A
- added U5: RT9193-15GB, RT9193:RT9193-33GB
- added U6: RT9193-28GB, RT9193:RT9193-33GB
- added Y1: 40MHz/±10ppm, ECS-384-10-37-CKM-TR:ECS-384-10-37-CKM-TR
Connections:
- new net 1.8V: J3.10, U5.VOUT
- new net 2.8V: J3.11, J3.4, R16.1, U6.VOUT
- new net 3.3V: U1.VDD3P3_CPU, U1.VDD3P3_RTC, U1.VDDA1, U1.VDDA2, U3.VDD, U3.VREGIN, U5.VIN, U6.VIN
- new net 5V: U$1.CE, U$1.VCC
- new net D+: J2.DP1, J2.DP2, U1.GPIO20
- new net D-: J2.DN1, J2.DN2, U1.GPIO19
- new net DTR: U3.DTR
- new net GND: AE1.FP, BTN1.I/O@2, C1.2, C2.2, C3.2, C4.2, C5.2, J1.GND_A, J1.GND_B, J1.SHIELD, J2.GND, J2.SHELL, J3.15, J3.SHLD@1, J3.SHLD@2, Q1.S1, R10.1, R15.1, R17.2, R6.2, R7.1, R8.1, R9.1, U$1.GND, U$1.TEMP, U1.GND, U2.GND, U3.GND, U5.GND, U6.GND, Y1.GND
- new net IO0: BTN2.I/O@1, R14.2, U1.GPIO0
- new net IO1: J3.3, U1.GPIO1
- new net IO2: J3.5, U1.GPIO2
- new net IO39: J3.19, U1.MTCK
- new net IO4: J3.20, U1.GPIO4
- new net IO40: J3.21, U1.MTDO
- new net IO41: J3.22, U1.MTDI
- new net IO42: J3.9, U1.MTMS
- new net IO45: J3.13, U1.GPIO45
- new net IO46: J3.14, U1.GPIO46
- new net IO48: J3.12, U1.SPICLK_N
- new net IO5: J3.17, U1.GPIO5
- new net IO6: J3.7, U1.GPIO6
- new net IO7: J3.18, U1.GPIO7
- new net IO8: J3.16, U1.GPIO8
- new net N$1: U1.SPICS0, U2./CS
- new net N$10: R4.2, U1.SPIQ
- new net N$11: R5.2, U1.SPID
- new net N$12: L1.2, U1.XTAL_P
- new net N$13: C2.1, L1.1, Y1.IN/OUT
- new net N$14: C1.1, U1.XTAL_N, Y1.OUT/IN
- new net N$15: BTN2.I/O@2, R6.1
- new net N$16: J2.CC1, R8.2
- new net N$17: J2.CC2, R7.2
- new net N$18: J2.VBUS
- new net N$19: J1.CC1, R9.2
- new net N$2: R1.1, U2./HOLD/RESET(IO3)
- new net N$20: J1.CC2, R10.2
- new net N$21: R11.2, U3.RXD
- new net N$22: U3.!SUSPENDB
- new net N$23: R12.2, U3.TXD
- new net N$24: U3.!RST
- new net N$25: U1.XTAL_32K_P
- new net N$26: C5.1, L2.2, U1.LNA_IN
- new net N$27: AE1.GND, C4.1, L2.1, L3.1
- new net N$28: C3.1, L3.2
- new net N$29: U1.XTAL_32K_N
- new net N$3: R1.2, U1.SPIHD
- new net N$30: U1.VDD3P3
- new net N$31: J3.6, R16.2
- new net N$32: J3.8, R15.2
- new net N$33: U1.U0TXD
- new net N$34: U3.VBUS
- new net N$35: R13.1
- new net N$36: R14.1
- new net N$39: U$1.BAT
- new net N$4: R2.1, U2./WP(IO2)
- new net N$40: U$1.PROG
- new net N$41: Q1.S2, U4.GND
- new net N$42: Q1.G1, U4.OC
- new net N$43: Q1.G2, U4.OD
- new net N$44: U4.CS
- new net N$45: U4.VCC
- new net N$46: U5.BP
- new net N$47: U6.BP
- new net N$48: J3.2, R17.1
- new net N$49: U5.EN
- new net N$5: R2.2, U1.SPIWP
- new net N$51: U6.EN
- new net N$6: R3.1, U2.CLK
- new net N$7: R4.1, U2.DO(IO1)
- new net N$8: R5.1, U2.DI(IO0)
- new net N$9: R3.2, U1.SPICLK
- new net RESET: BTN1.I/O@1, R13.2, U1.CHIP_PU
- new net RTS: U3.RTS
- new net RXD: R12.1, U1.U0RXD
- new net TXD: R11.1
- new net USB_D+: J1.DP1, J1.DP2, U3.D+
- new net USB_D-: J1.DN1, J1.DN2, U3.D-
- new net VDD_SPI: U1.VDD_SPI, U2.VCC
- new net V_USB: J1.VBUS_A, J1.VBUS_B
Other:
- note added: "0.1uF"
- note added: "1.2-10kohm arasında 1.2k : 1A 10k : 0.13A"
- note added: "100k"
- note added: "100ohm"
- note added: "10Kohm"
- note added: "10k ohm(NC)"
- note added: "10nF"
- note added: "10uF"
- note added: "10uF/25v"
- note added: "1K ohm"
- note added: "1N5819HW-7-F"
- note added: "1N5819HW-7-F 0.32-0.45v arası voltaj düşümü yapıyor"
- note added: "1kohm"
- note added: "1uF"
- note added: "1uF 16v"
- note added: "22.1k"
- note added: "22nF"
- note added: "2nH(0.1nH)"
- note added: "3.7v"
- note added: "47.5k"
- note added: "499ohm"
- note added: "Auto Program DTR RTS --> EN IO0 IO2 1 1 1 1 1 0 0 1 1 1 1 0 0 1 1 0 1 1 0 0"
- note added: "CAM_ENABLE"
- note added: "CAM_HREF"
- note added: "CAM_PCLK"
- note added: "CAM_PWDN"
- note added: "CAM_RST"
- note added: "CAM_SCL"
- note added: "CAM_SDA"
- note added: "CAM_VSYNC"
- note added: "CAM_XMCLK"
- note added: "CAM_Y2"
- note added: "CAM_Y3"
- note added: "CAM_Y4"
- note added: "CAM_Y5"
- note added: "CAM_Y6"
- note added: "CAM_Y7"
- note added: "CAM_Y8"
- note added: "CAM_Y9"
- note added: "Eğer J1 ve J2 connect edilirse sadece J1 den akım geçsin. J2 boş olsun"
- note added: "L8050QLT1G"
- note added: "Li-ion battery connector"
- note added: "RTC Sleep clock"
- note added: "SCH_ESP32-S3-DEVKITC-1_V1_20210312C.pdf: 10Kohm"
- note added: "capacitor: pros3 1uF"
- note added: "firebeetle 4.7 uF"
- note added: "firebeetle da 4.7uF 0.1uF kullanmış"
- note added: "firebeetle da 4.7uF 0.1uF kullanmış Ben önceki devremde 1uF 1uF 0.1uF kullanmışım"
- note added: "p channel mosfet"
- note added: "pull up resistor: 100k ohm in pros3"
- note added: "use a gpio pin to enable these regulators as enable pin"
