File: G0.sch (EAGLE design)
At the start: 48 parts, among them J1 USB4080-03-A_REVA1, J2 USB4085-GF-A_REVB, J3 SFV24R-3STBE1HLF, K1 112J-TDAR-R01, Q1 FS8205A, U1 ESP32-S3R8, U2 W25Q128JVSIQ, U3 CP2102N-A01-GQFN28, U4 DW01A, U5 RT9193-15GB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

Commit message: Rev1
Parts:
- removed C5: 12pF, SparkFun-Capacitors:0.1UF-0402-16V-10%
- removed L3: 0.8nH, SparkFun-Coils:INDUCTOR-0603-15NH
- added R22, R23: 0, SparkFun-Resistors:0OHM-0603-1/10W
- C3: value 5.6pF -> 1.5pF/±0.1; device SparkFun-Capacitors:0.1UF-0603-100V-10% -> SparkFun-Capacitors:0.22UF-0603-25V-10%
- C4: value 10pF -> 1.5pF/±0.1; device SparkFun-Capacitors:1.0UF-0805-25V-10% -> SparkFun-Capacitors:0.22UF-0603-25V-10%
- L2: value 0.8nH -> 2.7nH/±0.3; device SparkFun-Coils:INDUCTOR-0603-15NH -> SparkFun-Coils:INDUCTOR-0402-3.9NH
Connections:
- new net N$25: K1.6-VSS, K1.SW-B/GND, R22.2
- net GND: now also R22.1; no longer C5.2, K1.6-VSS, K1.SW-B/GND
- net N$26: now also C4.1; no longer C5.1
- net N$27: now also C3.1, R23.2; no longer AE1.GND, C4.1, L3.1
- net N$28: now also AE1.GND, R23.1; no longer C3.1, L3.2
Other:
- moved on the sheet: AE1, C3, C4, L2, R18, R19, R20, R21
