File: G0.sch (EAGLE design)
At the start: 39 parts, among them J1 USB4085-GF-A_REVB, J3 SFV24R-3STBE1HLF, K1 112J-TDAR-R01, Q1 FS8205A, U1 ESP32-S3R8, U2 W25Q128JVSIQ, U4 DW01A, U5 RT9193-15GB, U6 RT9193-28GB, Y1 40MHz/±10ppm/>500mV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

Commit message: first
Parts:
- removed SR4W035: (no value), SR4W035:SR4W035
- added ANT1: SR4W035, SR4W035:SR4W035
Connections:
- removed net N$26: GJM1555C1H1R5CB01D.1, LQW18AN2N2D00D.1, SR4W035.FEED
- removed net N$27: GJM1555C1H1R5CB01D.2, U1.LNA_IN
- new net N$20: GJM1555C1H1R5CB01D.1, U1.LNA_IN
- new net N$22: ANT1.FEED, GJM1555C1H1R5CB01D.2, LQW18AN2N2D00D.1
- net GND: now also ANT1.GND@1, ANT1.GND@2, ANT1.GND@3; no longer SR4W035.GND@1, SR4W035.GND@2, SR4W035.GND@3
Other:
- moved on the sheet: C1, C2, GJM1555C1H1R5CB01D, J1, LQW18AN2N2D00D, R7, R8, Y1
