File: G0 with UART.sch (EAGLE design)
At the start: 39 parts, among them J1 USB4085-GF-A_REVB, J3 SFV24R-3STBE1HLF, K1 112J-TDAR-R01, Q1 FS8205A, U1 ESP32-S3R8, U2 W25Q128JVSIQ, U4 DW01A, U5 RT9193-15GB, U6 RT9193-28GB, Y1 40MHz/±10ppm/>500mV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

Commit message: G0
Parts:
- removed SR4W035: (no value), SR4W035:SR4W035
- added J2: USB4085-GF-A_REVB, USB4085-GF-A_REVB:USB4085-GF-A_REVB
- added R10: 5.1k, SparkFun-Resistors:5.1KOHM5.1KOHM-0603-1/10W-1%
- added R11, R12, R13, R14: 0, SparkFun-Resistors:0OHM-0603-1/10W
- added U$2: (no value), SR4W035:SR4W035
- added U3: CP2102N-A01-GQFN28, CP2102N-A01-GQFN28:CP2102N-A01-GQFN28
- J1: value USB4085-GF-A_REVB -> USB4080-03-A_REVA1; device USB4085-GF-A_REVB:USB4085-GF-A_REVB -> USB4080-03-A_REVA1:USB4080-03-A_REVA1
- Y1: value 40MHz/±10ppm/>500mV -> 40MHz/±10ppm
Connections:
- removed net RX: U1.U0RXD
- new net DTR: U3.DTR
- new net N$19: J1.CC1, R9.2
- new net N$20: J1.CC2, R10.2
- new net N$21: R11.2, U3.RXD
- new net N$22: U3.!SUSPENDB
- new net N$23: R12.2, U3.TXD
- new net N$24: U3.!RST
- new net N$25: K1.6-VSS, K1.SW-B/GND, R22.2
- new net N$34: U3.VBUS
- new net N$35: R13.1
- new net N$36: R14.1
- new net RTS: U3.RTS
- new net RXD: R12.1, U1.U0RXD
- new net TXD: R11.1
- new net USB_D+: J1.DP1, J1.DP2, U3.D+
- new net USB_D-: J1.DN1, J1.DN2, U3.D-
- new net V_USB: J1.VBUS_A, J1.VBUS_B
- net 3.3V: now also U3.VDD, U3.VREGIN; no longer R9.2
- net 5V: no longer J1.VBUS
- net D+: now also J2.DP1, J2.DP2; no longer J1.DP1, J1.DP2
- net D-: now also J2.DN1, J2.DN2; no longer J1.DN1, J1.DN2
- net GND: now also J1.GND_A, J1.GND_B, J1.SHIELD, J2.GND, J2.SHELL, R10.1, R22.1, R9.1, U$2.GND@1, U$2.GND@2, U$2.GND@3, U3.GND; no longer J1.GND, J1.SHELL, R22.2, SR4W035.GND@1, SR4W035.GND@2, SR4W035.GND@3
- net IO0: now also R14.2
- net N$16: now also J2.CC1; no longer J1.CC1
- net N$17: now also J2.CC2; no longer J1.CC2
- net N$18: now also J2.VBUS; no longer K1.6-VSS, K1.SW-B/GND, R22.1
- net N$26: now also U$2.FEED; no longer SR4W035.FEED
- net RESET: now also R13.2; no longer R9.1
Other:
- note added: "10Kohm"
- note added: "10k ohm(NC)"
- note added: "10uF/25v"
- note added: "1K ohm"
- note added: "1uF 16v"
- note added: "22.1k"
- note added: "47.5k"
- note added: "499ohm"
- note added: "Auto Program DTR RTS --> EN IO0 IO2 1 1 1 1 1 0 0 1 1 1 1 0 0 1 1 0 1 1 0 0"
- note added: "Eğer J1 ve J2 connect edilirse sadece J1 den akım geçsin. J2 boş olsun"
- note added: "L8050QLT1G"
- note added: "TVS Diode"
- note added: "bidirectional diode"
- note removed: "499 ohm"
- note removed: "CL = (C1 × C4) / (C1 + C4) + Cstray"
- moved on the sheet: GJM1555C1H1R5CB01D, LQW18AN2N2D00D, Q1, R18, R19, R20, R21, R22, R7, R8, R9, U$1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
